Commit message: FIXED wrong xacro header definition

File: common_sensors/urdf/sensors/hokuyo_04lx_laser.gazebo.xacro (robot description, xacro)
@@ -1,5 +1,5 @@
 <?xml version="1.0"?>
 <root
-      xmlns:xacro="http://ros.org/wiki/xacro">
+      xmlns:xacro="http://www.ros.org/wiki/xacro">
   <xacro:macro name="hokuyo_04lx_laser_gazebo" params="name ros_topic update_rate min_angle max_angle">
     <gazebo reference="${name}_link">

File: common_sensors/urdf/sensors/hokuyo_04lx_laser.urdf.xacro (robot description, xacro)
@@ -3,5 +3,5 @@
       xmlns:controller="http://playerstage.sourceforge.net/gazebo/xmlschema/#controller"
       xmlns:interface="http://playerstage.sourceforge.net/gazebo/xmlschema/#interface"
-      xmlns:xacro="http://ros.org/wiki/xacro">
+      xmlns:xacro="http://www.ros.org/wiki/xacro">
   <xacro:include filename="$(find common_sensors)/urdf/sensors/hokuyo_04lx_laser.gazebo.xacro" />
   <xacro:macro name="hokuyo_04lx_laser" params="name parent *origin ros_topic update_rate min_angle max_angle">

File: common_sensors/urdf/sensors/hokuyo_utm30lx.urdf.xacro (robot description, xacro)
@@ -1,4 +1,4 @@
 <?xml version="1.0"?>
-<robot xmlns:xacro="http://ros.org/wiki/xacro">
+<robot xmlns:xacro="http://www.ros.org/wiki/xacro">
 <xacro:macro name="hokuyo_utm30lx" params="name parent *origin ros_topic update_rate ray_count min_angle max_angle">
 	<joint name="${name}_joint" type="fixed">

File: common_sensors/urdf/sensors/kinect.urdf.xacro (robot description, xacro)
@@ -1,4 +1,4 @@
 <?xml version="1.0"?>
-<root name="sensor_kinect" xmlns:xacro="http://ros.org/wiki/xacro">
+<root name="sensor_kinect" xmlns:xacro="http://www.ros.org/wiki/xacro">
 	<xacro:include filename="$(find common_sensors)/urdf/sensors/kinect_gazebo.xacro" />
         <xacro:include filename="$(find common_sensors)/urdf/sensors/kinect_properties.urdf.xacro"/>

File: common_sensors/urdf/sensors/kinect2.urdf.xacro (robot description, xacro)
@@ -1,4 +1,4 @@
 <?xml version="1.0"?>
-<robot xmlns:xacro="http://ros.org/wiki/xacro">
+<robot xmlns:xacro="http://www.ros.org/wiki/xacro">
   <xacro:include filename="$(find common_sensors)/urdf/sensors/kinect2.gazebo.xacro" />
   <xacro:include filename="$(find common_sensors)/urdf/sensors/kinect2_properties.urdf.xacro" />
@@ -23,5 +23,5 @@
         <origin xyz="-0.102 -0.148 0" rpy="0 0 0"/>
         <geometry>
-          <mesh filename="package://common_sensors/meshes/sensors/kinect2_assembly.STL" scale="0.001 0.001 0.001" />
+          <mesh filename="package://common_sensors/meshes/sensors/kinect2_assembly2.STL" scale="0.001 0.001 0.001" />
         </geometry>
         <material name="gray">
@@ -71,6 +71,15 @@
     </joint>
     <link name="${name}_kinect2_ir_optical_frame"/>
+    <!-- Add helper joint for correct position of skeleton tracking -->
+    <joint name="${name}_kinect2_tracker_frame_joint" type="fixed">
+      <origin xyz="0 0 0" rpy="0 0 3.141" />
+      <parent link="${name}_kinect2_ir_optical_frame"/>
+      <child link="${name}_kinect2_tracker_frame"/>
+    </joint>
+    <link name="${name}_kinect2_tracker_frame" />
     <!-- gazebo extensions -->
-    <xacro:kinect2_ir_gazebo link_name="${name}_kinect2_ir_link" frame_name="${name}_kinect2_ir_optical_frame" camera_name="head_mount_kinect2" />
+    <xacro:if value="$(arg kinect_sim)">
+        <xacro:kinect2_ir_gazebo link_name="${name}_kinect2_ir_link" frame_name="${name}_kinect2_ir_optical_frame" camera_name="${name}_ir" />
+    </xacro:if>
     <!-- kinect2 rgb sensor physical attachment -->
     <joint name="${name}_kinect2_rgb_joint" type="fixed">
@@ -110,5 +119,7 @@
     <link name="${name}_kinect2_rgb_optical_frame"/>
     <!-- gazebo extensions -->
-    <xacro:kinect2_rgb_gazebo link_name="${name}_kinect2_rgb_link" frame_name="${name}_kinect2_rgb_optical_frame" camera_name="head_mount_kinect2" />
+    <xacro:if value="$(arg kinect_sim)">
+        <xacro:kinect2_rgb_gazebo link_name="${name}_kinect2_rgb_link" frame_name="${name}_kinect2_rgb_optical_frame" camera_name="${name}_rgb" />
+    </xacro:if>
   </xacro:macro>
 </robot>

File: common_sensors/urdf/sensors/kinect_gazebo.xacro (robot description, xacro)
@@ -1,4 +1,4 @@
 <?xml version="1.0"?>
-<root name="kinect_gazebo" xmlns:xacro="http://ros.org/wiki/xacro">
+<root name="kinect_gazebo" xmlns:xacro="http://www.ros.org/wiki/xacro">
   <!-- Microsoft Kinect / ASUS Xtion PRO Live for simulation -->
   <xacro:include filename="$(find common_sensors)/urdf/common_properties.urdf.xacro" />

File: common_sensors/urdf/sensors/xtion.urdf.xacro (robot description, xacro)
@@ -1,4 +1,4 @@
 <?xml version="1.0"?>
-<robot name="sensor_asus_xtion_pro" xmlns:xacro="http://ros.org/wiki/xacro">
+<robot name="sensor_asus_xtion_pro" xmlns:xacro="http://www.ros.org/wiki/xacro">
 	<xacro:include filename="$(find common_sensors)/urdf/sensors/xtion_gazebo.urdf.xacro"/>
 	<!-- Xacro properties -->

File: common_sensors/urdf/sensors/xtion_gazebo.urdf.xacro (robot description, xacro)
@@ -1,4 +1,4 @@
 <?xml version="1.0"?>
-<robot name="xtion_gazebo" xmlns:xacro="http://ros.org/wiki/xacro">
+<robot name="xtion_gazebo" xmlns:xacro="http://www.ros.org/wiki/xacro">
   <!-- Microsoft Kinect / ASUS Xtion PRO Live for simulation -->
   <xacro:macro name="xtion_sim_3dsensor" params="camera_name">

File: common_sensors/urdf/sensors/xtion_xtended_stand.urdf.xacro (robot description, xacro)
@@ -1,4 +1,4 @@
 <?xml version="1.0" ?>
-<robot name="xtion_stand" xmlns:xacro="http://ros.org/wiki/xacro">
+<robot name="xtion_stand" xmlns:xacro="http://www.ros.org/wiki/xacro">
 	<xacro:include filename="$(find common_sensors)/urdf/sensors/xtion.urdf.xacro"/>
 	<xacro:macro name="xtion_standoff" params="parent number x_loc y_loc z_loc height">
